File: Trainiiii_Cape/Trainiiii_Cape.sch (EAGLE design)
At the start: 24 parts, among them J1 455-1750-1-ND, J2 455-1750-1-ND, Q1 220mA/50V/3.5Ω, Q2 220mA/50V/3.5Ω

Commit message: Organization and pin changes.
Moved ultrasonic lines to pins that don't interfere with BBB boot sequence. Began organizing things into sheets!
Parts:
- added J3: (no value), SparkFun-Connectors:CONN_02
- added U1: AP1509-50, RoboJackets-PowerICs:AP1509-50
Connections:
- new net POWER_BUTTON: B1P9.PWR_BUT, J3.2
- net 5V: now also B1P9.VDD_5V@1, B1P9.VDD_5V@2; no longer B1P9.SYS_5V@1, B1P9.SYS_5V@2
- net GND: now also J3.1, U1.GND, U1.SD
- net US_ECHO_3V3: now also B1P8.GPIO_27; no longer B1P8.GPIO_71
- net US_TRIGGER_3V3: now also B1P8.GPIO_47; no longer B1P8.GPIO_70
- net V_BATT: now also U1.VIN
Other:
- note added: "BeagleBone Black Cape Connectors"
- note added: "Encoders"
- note added: "Line Sensors"
- note added: "Motors"
- note added: "Power Management"
- note added: "Sensors"
- note added: "Ultrasonic Sensor"
